File: mod-dac.sch (KiCad schematic (older format))
At the start: 9 parts, among them U1 TL072

Commit message: looking like the right values for ~4x gain
Parts:
- R1: value 20k -> 23.7k
- R2: value 130k -> 100k
- V1: Spice_Model dc 0 ac 0 sin(1.25 1.25 200) -> dc 1.25 ac 1.25 sin(1.25 1.25 100)
- V2: Spice_Model dc 1.087 ac 0 -> dc 1 ac 0
Other:
- note added: ".ac dec 1000 100 20000"
Changed lines of the file:
@@
 P 3225 1950
 F 0 "R1" V 3018 1950 50  0000 C CNN
-F 1 "20k" V 3109 1950 50  0000 C CNN
+F 1 "23.7k" V 3109 1950 50  0000 C CNN
 F 2 "" V 3155 1950 50  0001 C CNN
 F 3 "~" H 3225 1950 50  0001 C CNN
@@
 F 3 "" H 2475 2275 50  0001 C CNN
 F 4 "V" H 2475 2275 50  0001 C CNN "Spice_Primitive"
-F 5 "dc 0 ac 0 sin(1.25 1.25 200)" H 2475 2275 50  0001 C CNN "Spice_Model"
+F 5 "dc 1.25 ac 1.25 sin(1.25 1.25 100)" H 2475 2275 50  0001 C CNN "Spice_Model"
 F 6 "Y" H 2475 2275 50  0001 C CNN "Spice_Netlist_Enabled"
 	1    2475 2275
@@
 P 3825 975
 F 0 "R2" V 4032 975 50  0000 C CNN
-F 1 "130k" V 3941 975 50  0000 C CNN
+F 1 "100k" V 3941 975 50  0000 C CNN
 F 2 "" V 3755 975 50  0001 C CNN
 F 3 "~" H 3825 975 50  0001 C CNN
@@
 F 3 "" H 3425 2600 50  0001 C CNN
 F 4 "V" H 3425 2600 50  0001 C CNN "Spice_Primitive"
-F 5 "dc 1.087 ac 0" H 3425 2600 50  0001 C CNN "Spice_Model"
+F 5 "dc 1 ac 0" H 3425 2600 50  0001 C CNN "Spice_Model"
 F 6 "Y" H 3425 2600 50  0001 C CNN "Spice_Netlist_Enabled"
 	1    3425 2600
@@
 Wire Wire Line
 	6000 1550 6000 1900
+Text Notes 875  4075 0    50   ~ 0
+.ac dec 1000 100 20000
 $EndSCHEMATC

Commit message: updated with TL074
Parts:
- removed U1: TL072, symbol Amplifier_Operational:TL072
- added U1: TL074, symbol Amplifier_Operational:TL074
Changed lines of the file:
@@
 Wire Wire Line
 	2850 1950 2475 1950
-$Comp
-L Amplifier_Operational:TL072 U1
-U 1 1 5C2187D4
-P 3825 2050
-F 0 "U1" H 3825 1683 50  0000 C CNN
-F 1 "TL072" H 3825 1774 50  0000 C CNN
-F 2 "" H 3825 2050 50  0001 C CNN
-F 3 "http://www.ti.com/lit/ds/symlink/tl071.pdf" H 3825 2050 50  0001 C CNN
-F 4 "X" H 3825 2050 50  0001 C CNN "Spice_Primitive"
-F 5 "TL072" H 3825 2050 50  0001 C CNN "Spice_Model"
-F 6 "Y" H 3825 2050 50  0001 C CNN "Spice_Netlist_Enabled"
-F 7 "TL072.301" H 3825 2050 50  0001 C CNN "Spice_Lib_File"
-F 8 "3 2 8 4 1" H 3825 2050 50  0001 C CNN "Spice_Node_Sequence"
-	1    3825 2050
-	1    0    0    1
-$EndComp
-$Comp
-L Amplifier_Operational:TL072 U1
-U 3 1 5C21887F
-P 6100 2200
-F 0 "U1" H 6058 2246 50  0000 L CNN
-F 1 "TL072" H 6058 2155 50  0000 L CNN
-F 2 "" H 6100 2200 50  0001 C CNN
-F 3 "http://www.ti.com/lit/ds/symlink/tl071.pdf" H 6100 2200 50  0001 C CNN
-	3    6100 2200
-	1    0    0    -1
-$EndComp
 Text GLabel 5025 2050 2    50   Input ~ 0
 vout
@@
 Text Notes 875  4075 0    50   ~ 0
 .ac dec 1000 100 20000
+$Comp
+L Amplifier_Operational:TL074 U1
+U 1 1 5C2693FF
+P 3825 2050
+F 0 "U1" H 3825 1683 50  0000 C CNN
+F 1 "TL074" H 3825 1774 50  0000 C CNN
+F 2 "" H 3775 2150 50  0001 C CNN
+F 3 "http://www.ti.com/lit/ds/symlink/tl071.pdf" H 3875 2250 50  0001 C CNN
+F 4 "X" H 3825 2050 50  0001 C CNN "Spice_Primitive"
+F 5 "TL074" H 3825 2050 50  0001 C CNN "Spice_Model"
+F 6 "Y" H 3825 2050 50  0001 C CNN "Spice_Netlist_Enabled"
+F 7 "3 2 4 11 1" H 3825 2050 50  0001 C CNN "Spice_Node_Sequence"
+F 8 "TL074.301" H 3825 2050 50  0001 C CNN "Spice_Lib_File"
+	1    3825 2050
+	1    0    0    1
+$EndComp
+$Comp
+L Amplifier_Operational:TL074 U1
+U 5 1 5C2694AE
+P 6100 2200
+F 0 "U1" H 6058 2246 50  0000 L CNN
+F 1 "TL074" H 6058 2155 50  0000 L CNN
+F 2 "" H 6050 2300 50  0001 C CNN
+F 3 "http://www.ti.com/lit/ds/symlink/tl071.pdf" H 6150 2400 50  0001 C CNN
+	5    6100 2200
+	1    0    0    -1
+$EndComp
 $EndSCHEMATC

Commit message: major schematic progress
Parts:
- removed C1: 100pF, symbol Device:C
- removed R1: 23.7k, symbol Device:R
- removed R2: 100k, symbol Device:R
- removed R3: 1k, symbol Device:R
- removed U1: TL074, symbol Amplifier_Operational:TL074
- removed V1: VOLTAGE, symbol pspice:VSOURCE
- removed V2, V3, V4: VSOURCE, symbol pspice:VSOURCE
- added C13: 22u, symbol Device:C
- added C14, C15, C16: 1u, symbol Device:C
- added J1: digi in, symbol Connector_Generic:Conn_01x04
- added J2: cv out, symbol Connector_Generic:Conn_01x09
- added TR1: VREF TRIM, symbol trim:TRIM
- added TR2: BIAS TRIM, symbol trim:TRIM
- added U4: DAC8168, symbol xnorman:DAC8168
Connections:
- net labels added: +3.3V, DIN, REFVCC, SCLK, \SYNC, dac0, dac1, dac2, dac3, dac4, dac5, dac6, dac7, vout0, vout1, vout2, vout3, vout4, vout5, vout6, vout7, vref
- net labels removed: vin, vinv, vopout, vout
- wire segments 31 -> 51
Other:
- note added: "do we want a separate vreg for the reference voltages?"
- note removed: ".ac dec 1000 100 20000"

Commit message: added 15v power
Parts:
- added C17, C18: 10uF, Capacitors_THT:CP_Radial_D7.5mm_P2.50mm, symbol shift-triggers-rescue:CP
- added P1: MTA-156-4, mta-156:MTA-156-4, symbol shift-triggers-rescue:MTA-156-4
- added R25, R26: bead, Resistors_THT:R_Axial_DIN0207_L6.3mm_D2.5mm_P10.16mm_Horizontal, symbol shift-triggers-rescue:R
Connections:
- net labels added: +15V, -15V
- wire segments 51 -> 72
Changed lines of the file:
@@
 EESchema Schematic File Version 4
 LIBS:mod-dac-cache
+LIBS:shift-triggers-cache
 EELAYER 26 0
 EELAYER END
@@
 Wire Wire Line
 	1150 2900 1075 2900
+$Comp
+L shift-triggers-rescue:R R26
+U 1 1 5C27DFC7
+P 7625 3775
+F 0 "R26" V 7705 3775 50  0000 C CNN
+F 1 "bead" V 7625 3775 50  0000 C CNN
+F 2 "Resistors_THT:R_Axial_DIN0207_L6.3mm_D2.5mm_P10.16mm_Horizontal" V 7555 3775 50  0001 C CNN
+F 3 "" H 7625 3775 50  0000 C CNN
+	1    7625 3775
+	0    -1   -1   0
+$EndComp
+$Comp
+L shift-triggers-rescue:CP C18
+U 1 1 5C27DFEA
+P 7875 4050
+F 0 "C18" H 7900 4150 50  0000 L CNN
+F 1 "10uF" H 7900 3950 50  0000 L CNN
+F 2 "Capacitors_THT:CP_Radial_D7.5mm_P2.50mm" H 7913 3900 50  0001 C CNN
+F 3 "" H 7875 4050 50  0000 C CNN
+	1    7875 4050
+	1    0    0    -1
+$EndComp
+$Comp
+L shift-triggers-rescue:MTA-156-4 P1
+U 1 1 5C27DFF1
+P 6900 3925
+F 0 "P1" H 6900 4175 50  0000 C CNN
+F 1 "MTA-156-4" V 7000 3925 50  0000 C CNN
+F 2 "mta-156:MTA-156-4" H 6900 3925 50  0001 C CNN
+F 3 "" H 6900 3925 50  0000 C CNN
+	1    6900 3925
+	-1   0    0    -1
+$EndComp
+Wire Wire Line
+	7475 3775 7100 3775
+Wire Wire Line
+	7775 3775 7875 3775
+Wire Wire Line
+	7875 3775 7875 3900
+$Comp
+L shift-triggers-rescue:GND #PWR016
+U 1 1 5C27E007
+P 7875 4250
+F 0 "#PWR016" H 7875 4000 50  0001 C CNN
+F 1 "GND" H 7875 4100 50  0000 C CNN
+F 2 "" H 7875 4250 50  0000 C CNN
+F 3 "" H 7875 4250 50  0000 C CNN
+	1    7875 4250
+	1    0    0    -1
+$EndComp
+Wire Wire Line
+	7875 4200 7875 4225
+Wire Wire Line
+	7100 3875 7500 3875
+Wire Wire Line
+	7500 3875 7500 3975
+Wire Wire Line
+	7500 3975 7100 3975
+Wire Wire Line
+	7500 4225 7625 4225
+Connection ~ 7875 4225
+Connection ~ 7500 3975
+$Comp
+L shift-triggers-rescue:PWR_FLAG #FLG01
+U 1 1 5C27E01D
+P 8225 4250
+F 0 "#FLG01" H 8225 4325 50  0001 C CNN
+F 1 "PWR_FLAG" H 8225 4400 50  0000 C CNN
+F 2 "" H 8225 4250 50  0001 C CNN
+F 3 "" H 8225 4250 50  0001 C CNN
+	1    8225 4250
+	-1   0    0    1
+$EndComp
+Wire Wire Line
+	7875 4225 7875 4250
+Wire Wire Line
+	7500 3975 7500 4225
+$Comp
+L shift-triggers-rescue:R R25
+U 1 1 5C2844C4
+P 7300 4225
+F 0 "R25" V 7380 4225 50  0000 C CNN
+F 1 "bead" V 7300 4225 50  0000 C CNN
+F 2 "Resistors_THT:R_Axial_DIN0207_L6.3mm_D2.5mm_P10.16mm_Horizontal" V 7230 4225 50  0001 C CNN
+F 3 "" H 7300 4225 50  0000 C CNN
+	1    7300 4225
+	1    0    0    -1
+$EndComp
+Wire Wire Line
+	7300 4075 7100 4075
+$Comp
+L shift-triggers-rescue:CP C17
+U 1 1 5C285D73
+P 7625 4375
+F 0 "C17" H 7650 4475 50  0000 L CNN
+F 1 "10uF" H 7650 4275 50  0000 L CNN
+F 2 "Capacitors_THT:CP_Radial_D7.5mm_P2.50mm" H 7663 4225 50  0001 C CNN
+F 3 "" H 7625 4375 50  0000 C CNN
+	1    7625 4375
+	1    0    0    -1
+$EndComp
+Connection ~ 7625 4225
+Wire Wire Line
+	7625 4225 7875 4225
+Wire Wire Line
+	7300 4375 7300 4525
+Wire Wire Line
+	7300 4525 7475 4525
+Wire Wire Line
+	7875 4225 8225 4225
+Wire Wire Line
+	8225 4225 8225 4250
+$Comp
+L power:+15V #PWR015
+U 1 1 5C2937C8
+P 7875 3550
+F 0 "#PWR015" H 7875 3400 50  0001 C CNN
+F 1 "+15V" H 7890 3723 50  0000 C CNN
+F 2 "" H 7875 3550 50  0001 C CNN
+F 3 "" H 7875 3550 50  0001 C CNN
+	1    7875 3550
+	1    0    0    -1
+$EndComp
+$Comp
+L power:-15V #PWR014
+U 1 1 5C293829
+P 7475 4625
+F 0 "#PWR014" H 7475 4725 50  0001 C CNN
+F 1 "-15V" H 7490 4798 50  0000 C CNN
+F 2 "" H 7475 4625 50  0001 C CNN
+F 3 "" H 7475 4625 50  0001 C CNN
+	1    7475 4625
+	-1   0    0    1
+$EndComp
+Wire Wire Line
+	7475 4525 7475 4625
+Connection ~ 7475 4525
+Wire Wire Line
+	7475 4525 7625 4525
+Wire Wire Line
+	7875 3550 7875 3775
+Connection ~ 7875 3775
+$Comp
+L shift-triggers-rescue:PWR_FLAG #FLG0101
+U 1 1 5C298F27
+P 7225 4525
+F 0 "#FLG0101" H 7225 4600 50  0001 C CNN
+F 1 "PWR_FLAG" H 7225 4675 50  0000 C CNN
+F 2 "" H 7225 4525 50  0001 C CNN
+F 3 "" H 7225 4525 50  0001 C CNN
+	1    7225 4525
+	0    -1   -1   0
+$EndComp
+Wire Wire Line
+	7225 4525 7300 4525
+Connection ~ 7300 4525
+$Comp
+L shift-triggers-rescue:PWR_FLAG #FLG0102
+U 1 1 5C29A528
+P 8175 3775
+F 0 "#FLG0102" H 8175 3850 50  0001 C CNN
+F 1 "PWR_FLAG" H 8175 3925 50  0000 C CNN
+F 2 "" H 8175 3775 50  0001 C CNN
+F 3 "" H 8175 3775 50  0001 C CNN
+	1    8175 3775
+	0    1    1    0
+$EndComp
+Wire Wire Line
+	7875 3775 8175 3775
 $EndSCHEMATC
