File: mod-dac.sch (KiCad schematic (older format))
At the start: 14 parts, among them J1 digi in, J2 cv out, P1 MTA-156-4, U4 DAC8168

Commit message: fixed up power supply
Parts:
- removed C17, C18: 10uF, Capacitors_THT:CP_Radial_D7.5mm_P2.50mm, symbol shift-triggers-rescue:CP
- removed P1: MTA-156-4, mta-156:MTA-156-4, symbol shift-triggers-rescue:MTA-156-4
- removed R25, R26: bead, Resistors_THT:R_Axial_DIN0207_L6.3mm_D2.5mm_P10.16mm_Horizontal, symbol shift-triggers-rescue:R
- added C17, C18: 10uF, symbol Device:CP
- added L1, L2: Ferrite_Bead_Small, symbol Device:Ferrite_Bead_Small
- added P1: MTA-156-4, symbol mta-156:MTA-156-4
Connections:
- wire segments 72 -> 73
Changed lines of the file:
@@
 Wire Wire Line
 	1150 2900 1075 2900
-$Comp
-L shift-triggers-rescue:R R26
-U 1 1 5C27DFC7
-P 7625 3775
-F 0 "R26" V 7705 3775 50  0000 C CNN
-F 1 "bead" V 7625 3775 50  0000 C CNN
-F 2 "Resistors_THT:R_Axial_DIN0207_L6.3mm_D2.5mm_P10.16mm_Horizontal" V 7555 3775 50  0001 C CNN
-F 3 "" H 7625 3775 50  0000 C CNN
-	1    7625 3775
-	0    -1   -1   0
-$EndComp
-$Comp
-L shift-triggers-rescue:CP C18
-U 1 1 5C27DFEA
-P 7875 4050
-F 0 "C18" H 7900 4150 50  0000 L CNN
-F 1 "10uF" H 7900 3950 50  0000 L CNN
-F 2 "Capacitors_THT:CP_Radial_D7.5mm_P2.50mm" H 7913 3900 50  0001 C CNN
-F 3 "" H 7875 4050 50  0000 C CNN
-	1    7875 4050
-	1    0    0    -1
-$EndComp
-$Comp
-L shift-triggers-rescue:MTA-156-4 P1
-U 1 1 5C27DFF1
-P 6900 3925
-F 0 "P1" H 6900 4175 50  0000 C CNN
-F 1 "MTA-156-4" V 7000 3925 50  0000 C CNN
-F 2 "mta-156:MTA-156-4" H 6900 3925 50  0001 C CNN
-F 3 "" H 6900 3925 50  0000 C CNN
-	1    6900 3925
-	-1   0    0    -1
-$EndComp
 Wire Wire Line
-	7475 3775 7100 3775
+	7525 3775 7100 3775
 Wire Wire Line
-	7775 3775 7875 3775
-Wire Wire Line
-	7875 3775 7875 3900
-$Comp
-L shift-triggers-rescue:GND #PWR016
-U 1 1 5C27E007
-P 7875 4250
-F 0 "#PWR016" H 7875 4000 50  0001 C CNN
-F 1 "GND" H 7875 4100 50  0000 C CNN
-F 2 "" H 7875 4250 50  0000 C CNN
-F 3 "" H 7875 4250 50  0000 C CNN
-	1    7875 4250
-	1    0    0    -1
-$EndComp
-Wire Wire Line
-	7875 4200 7875 4225
+	7725 3775 8125 3775
 Wire Wire Line
 	7100 3875 7500 3875
 Wire Wire Line
-	7500 3875 7500 3975
+	7500 3875 7500 3950
 Wire Wire Line
 	7500 3975 7100 3975
 Wire Wire Line
-	7500 4225 7625 4225
-Connection ~ 7875 4225
-Connection ~ 7500 3975
-$Comp
-L shift-triggers-rescue:PWR_FLAG #FLG01
-U 1 1 5C27E01D
-P 8225 4250
-F 0 "#FLG01" H 8225 4325 50  0001 C CNN
-F 1 "PWR_FLAG" H 8225 4400 50  0000 C CNN
-F 2 "" H 8225 4250 50  0001 C CNN
-F 3 "" H 8225 4250 50  0001 C CNN
-	1    8225 4250
-	-1   0    0    1
-$EndComp
-Wire Wire Line
-	7875 4225 7875 4250
-Wire Wire Line
-	7500 3975 7500 4225
-$Comp
-L shift-triggers-rescue:R R25
-U 1 1 5C2844C4
-P 7300 4225
-F 0 "R25" V 7380 4225 50  0000 C CNN
-F 1 "bead" V 7300 4225 50  0000 C CNN
-F 2 "Resistors_THT:R_Axial_DIN0207_L6.3mm_D2.5mm_P10.16mm_Horizontal" V 7230 4225 50  0001 C CNN
-F 3 "" H 7300 4225 50  0000 C CNN
-	1    7300 4225
-	1    0    0    -1
-$EndComp
-Wire Wire Line
 	7300 4075 7100 4075
-$Comp
-L shift-triggers-rescue:CP C17
-U 1 1 5C285D73
-P 7625 4375
-F 0 "C17" H 7650 4475 50  0000 L CNN
-F 1 "10uF" H 7650 4275 50  0000 L CNN
-F 2 "Capacitors_THT:CP_Radial_D7.5mm_P2.50mm" H 7663 4225 50  0001 C CNN
-F 3 "" H 7625 4375 50  0000 C CNN
-	1    7625 4375
-	1    0    0    -1
-$EndComp
-Connection ~ 7625 4225
-Wire Wire Line
-	7625 4225 7875 4225
-Wire Wire Line
-	7300 4375 7300 4525
-Wire Wire Line
-	7300 4525 7475 4525
-Wire Wire Line
-	7875 4225 8225 4225
-Wire Wire Line
-	8225 4225 8225 4250
 $Comp
 L power:+15V #PWR015
 U 1 1 5C2937C8
-P 7875 3550
-F 0 "#PWR015" H 7875 3400 50  0001 C CNN
-F 1 "+15V" H 7890 3723 50  0000 C CNN
-F 2 "" H 7875 3550 50  0001 C CNN
-F 3 "" H 7875 3550 50  0001 C CNN
-	1    7875 3550
+P 8125 3550
+F 0 "#PWR015" H 8125 3400 50  0001 C CNN
+F 1 "+15V" H 8140 3723 50  0000 C CNN
+F 2 "" H 8125 3550 50  0001 C CNN
+F 3 "" H 8125 3550 50  0001 C CNN
+	1    8125 3550
 	1    0    0    -1
 $EndComp
@@
 L power:-15V #PWR014
 U 1 1 5C293829
-P 7475 4625
-F 0 "#PWR014" H 7475 4725 50  0001 C CNN
-F 1 "-15V" H 7490 4798 50  0000 C CNN
-F 2 "" H 7475 4625 50  0001 C CNN
-F 3 "" H 7475 4625 50  0001 C CNN
-	1    7475 4625
+P 7800 4750
+F 0 "#PWR014" H 7800 4850 50  0001 C CNN
+F 1 "-15V" H 7815 4923 50  0000 C CNN
+F 2 "" H 7800 4750 50  0001 C CNN
+F 3 "" H 7800 4750 50  0001 C CNN
+	1    7800 4750
 	-1   0    0    1
 $EndComp
 Wire Wire Line
-	7475 4525 7475 4625
-Connection ~ 7475 4525
-Wire Wire Line
-	7475 4525 7625 4525
-Wire Wire Line
-	7875 3550 7875 3775
-Connection ~ 7875 3775
+	8125 3550 8125 3775
 $Comp
-L shift-triggers-rescue:PWR_FLAG #FLG0101
-U 1 1 5C298F27
-P 7225 4525
-F 0 "#FLG0101" H 7225 4600 50  0001 C CNN
-F 1 "PWR_FLAG" H 7225 4675 50  0000 C CNN
-F 2 "" H 7225 4525 50  0001 C CNN
-F 3 "" H 7225 4525 50  0001 C CNN
-	1    7225 4525
-	0    -1   -1   0
+L Device:Ferrite_Bead_Small L2
+U 1 1 5C27B7E6
+P 7625 3775
+F 0 "L2" V 7388 3775 50  0000 C CNN
+F 1 "Ferrite_Bead_Small" V 7479 3775 50  0000 C CNN
+F 2 "" V 7555 3775 50  0001 C CNN
+F 3 "~" H 7625 3775 50  0001 C CNN
+	1    7625 3775
+	0    1    1    0
+$EndComp
+$Comp
+L Device:Ferrite_Bead_Small L1
+U 1 1 5C27B88B
+P 7400 4500
+F 0 "L1" V 7163 4500 50  0000 C CNN
+F 1 "Ferrite_Bead_Small" V 7254 4500 50  0000 C CNN
+F 2 "" V 7330 4500 50  0001 C CNN
+F 3 "~" H 7400 4500 50  0001 C CNN
+	1    7400 4500
+	0    1    1    0
+$EndComp
+$Comp
+L mta-156:MTA-156-4 P1
+U 1 1 5C27B987
+P 6900 3925
+F 0 "P1" H 6819 4290 50  0000 C CNN
+F 1 "MTA-156-4" H 6819 4199 50  0000 C CNN
+F 2 "" H 6900 3925 50  0000 C CNN
+F 3 "" H 6900 3925 50  0000 C CNN
+	1    6900 3925
+	-1   0    0    -1
+$EndComp
+$Comp
+L Device:CP C18
+U 1 1 5C28145A
+P 8300 3925
+F 0 "C18" H 8418 3971 50  0000 L CNN
+F 1 "10uF" H 8418 3880 50  0000 L CNN
+F 2 "" H 8338 3775 50  0001 C CNN
+F 3 "~" H 8300 3925 50  0001 C CNN
+	1    8300 3925
+	1    0    0    -1
+$EndComp
+$Comp
+L Device:CP C17
+U 1 1 5C2814BB
+P 8075 4650
+F 0 "C17" H 8193 4696 50  0000 L CNN
+F 1 "10uF" H 8193 4605 50  0000 L CNN
+F 2 "" H 8113 4500 50  0001 C CNN
+F 3 "~" H 8075 4650 50  0001 C CNN
+	1    8075 4650
+	1    0    0    -1
 $EndComp
 Wire Wire Line
-	7225 4525 7300 4525
-Connection ~ 7300 4525
+	8125 3775 8250 3775
+Connection ~ 8125 3775
+Wire Wire Line
+	7500 4500 7800 4500
+Wire Wire Line
+	7800 4500 7800 4750
+Connection ~ 7800 4500
+Wire Wire Line
+	7800 4500 7950 4500
 $Comp
-L shift-triggers-rescue:PWR_FLAG #FLG0102
-U 1 1 5C29A528
-P 8175 3775
-F 0 "#FLG0102" H 8175 3850 50  0001 C CNN
-F 1 "PWR_FLAG" H 8175 3925 50  0000 C CNN
-F 2 "" H 8175 3775 50  0001 C CNN
-F 3 "" H 8175 3775 50  0001 C CNN
-	1    8175 3775
+L power:GND #PWR016
+U 1 1 5C2901E5
+P 7600 3950
+F 0 "#PWR016" H 7600 3700 50  0001 C CNN
+F 1 "GND" H 7605 3777 50  0000 C CNN
+F 2 "" H 7600 3950 50  0001 C CNN
+F 3 "" H 7600 3950 50  0001 C CNN
+	1    7600 3950
+	1    0    0    -1
+$EndComp
+Wire Wire Line
+	7600 3950 7500 3950
+Connection ~ 7500 3950
+Wire Wire Line
+	7500 3950 7500 3975
+$Comp
+L power:GND #PWR018
+U 1 1 5C29161E
+P 8300 4125
+F 0 "#PWR018" H 8300 3875 50  0001 C CNN
+F 1 "GND" H 8305 3952 50  0000 C CNN
+F 2 "" H 8300 4125 50  0001 C CNN
+F 3 "" H 8300 4125 50  0001 C CNN
+	1    8300 4125
+	1    0    0    -1
+$EndComp
+Wire Wire Line
+	8300 4075 8300 4125
+$Comp
+L power:GND #PWR017
+U 1 1 5C292A6F
+P 8075 4900
+F 0 "#PWR017" H 8075 4650 50  0001 C CNN
+F 1 "GND" H 8080 4727 50  0000 C CNN
+F 2 "" H 8075 4900 50  0001 C CNN
+F 3 "" H 8075 4900 50  0001 C CNN
+	1    8075 4900
+	1    0    0    -1
+$EndComp
+Wire Wire Line
+	8075 4800 8075 4900
+Wire Wire Line
+	7300 4075 7300 4500
+$Comp
+L power:PWR_FLAG #FLG0101
+U 1 1 5C2A6034
+P 7950 4425
+F 0 "#FLG0101" H 7950 4500 50  0001 C CNN
+F 1 "PWR_FLAG" H 7950 4599 50  0000 C CNN
+F 2 "" H 7950 4425 50  0001 C CNN
+F 3 "~" H 7950 4425 50  0001 C CNN
+	1    7950 4425
+	1    0    0    -1
+$EndComp
+$Comp
+L power:PWR_FLAG #FLG0102
+U 1 1 5C2A6062
+P 8375 3675
+F 0 "#FLG0102" H 8375 3750 50  0001 C CNN
+F 1 "PWR_FLAG" H 8375 3849 50  0000 C CNN
+F 2 "" H 8375 3675 50  0001 C CNN
+F 3 "~" H 8375 3675 50  0001 C CNN
+	1    8375 3675
+	1    0    0    -1
+$EndComp
+Wire Wire Line
+	8375 3675 8250 3675
+Wire Wire Line
+	8250 3675 8250 3775
+Connection ~ 8250 3775
+Wire Wire Line
+	8250 3775 8300 3775
+Wire Wire Line
+	7950 4425 7950 4500
+Connection ~ 7950 4500
+Wire Wire Line
+	7950 4500 8075 4500
+$Comp
+L power:PWR_FLAG #FLG0103
+U 1 1 5C2A8DC7
+P 7650 3875
+F 0 "#FLG0103" H 7650 3950 50  0001 C CNN
+F 1 "PWR_FLAG" V 7650 4003 50  0000 L CNN
+F 2 "" H 7650 3875 50  0001 C CNN
+F 3 "~" H 7650 3875 50  0001 C CNN
+	1    7650 3875
 	0    1    1    0
 $EndComp
 Wire Wire Line
-	7875 3775 8175 3775
+	7650 3875 7500 3875
+Connection ~ 7500 3875
 $EndSCHEMATC

Commit message: corrected cap orientation
Connections:
- wire segments 73 -> 74
Changed lines of the file:
@@
 L Device:CP C17
 U 1 1 5C2814BB
-P 8075 4650
-F 0 "C17" H 8193 4696 50  0000 L CNN
-F 1 "10uF" H 8193 4605 50  0000 L CNN
-F 2 "" H 8113 4500 50  0001 C CNN
-F 3 "~" H 8075 4650 50  0001 C CNN
-	1    8075 4650
-	1    0    0    -1
+P 8175 4700
+F 0 "C17" H 8293 4746 50  0000 L CNN
+F 1 "10uF" H 8293 4655 50  0000 L CNN
+F 2 "" H 8213 4550 50  0001 C CNN
+F 3 "~" H 8175 4700 50  0001 C CNN
+	1    8175 4700
+	-1   0    0    1
 $EndComp
 Wire Wire Line
@@
 L power:GND #PWR017
 U 1 1 5C292A6F
-P 8075 4900
-F 0 "#PWR017" H 8075 4650 50  0001 C CNN
-F 1 "GND" H 8080 4727 50  0000 C CNN
-F 2 "" H 8075 4900 50  0001 C CNN
-F 3 "" H 8075 4900 50  0001 C CNN
-	1    8075 4900
+P 8175 4925
+F 0 "#PWR017" H 8175 4675 50  0001 C CNN
+F 1 "GND" H 8180 4752 50  0000 C CNN
+F 2 "" H 8175 4925 50  0001 C CNN
+F 3 "" H 8175 4925 50  0001 C CNN
+	1    8175 4925
 	1    0    0    -1
 $EndComp
-Wire Wire Line
-	8075 4800 8075 4900
 Wire Wire Line
 	7300 4075 7300 4500
@@
 Wire Wire Line
 	7950 4425 7950 4500
-Connection ~ 7950 4500
-Wire Wire Line
-	7950 4500 8075 4500
 $Comp
 L power:PWR_FLAG #FLG0103
@@
 	7650 3875 7500 3875
 Connection ~ 7500 3875
+Wire Wire Line
+	7950 4500 8175 4500
+Wire Wire Line
+	8175 4500 8175 4550
+Connection ~ 7950 4500
+Wire Wire Line
+	8175 4850 8175 4925
 $EndSCHEMATC

Commit message: 3.3v supply, also.. updated per stages
Parts:
- added C19, C20, C21, C22: 22uF, symbol Device:CP
- added L3: BEAD, symbol Device:Ferrite_Bead_Small
- added U5: LD2981, symbol xnorman:LD2981
- C17, C18: value 10uF -> 22uF
- L1, L2: value Ferrite_Bead_Small -> BEAD
Connections:
- wire segments 74 -> 98

Commit message: removed polar parts
Parts:
- removed C17, C18, C19, C20, C21, C22: 22uF, symbol Device:CP
- added C17, C18, C19, C20, C21, C22: 22u, symbol Device:C
Changed lines of the file:
@@
 	-1   0    0    -1
-$EndComp
-$Comp
-L Device:CP C17
-U 1 1 5C2814BB
-P 8300 4300
-F 0 "C17" H 8418 4346 50  0000 L CNN
-F 1 "22uF" H 8418 4255 50  0000 L CNN
-F 2 "" H 8338 4150 50  0001 C CNN
-F 3 "~" H 8300 4300 50  0001 C CNN
-	1    8300 4300
-	1    0    0    -1
 $EndComp
 Wire Wire Line
@@
 Wire Wire Line
 	8400 2675 8475 2675
-$Comp
-L Device:CP C20
-U 1 1 5C2917BD
-P 8475 2850
-F 0 "C20" H 8593 2896 50  0000 L CNN
-F 1 "22uF" H 8593 2805 50  0000 L CNN
-F 2 "" H 8513 2700 50  0001 C CNN
-F 3 "~" H 8475 2850 50  0001 C CNN
-	1    8475 2850
-	1    0    0    -1
-$EndComp
 Wire Wire Line
 	8475 2675 8475 2700
@@
 Wire Wire Line
 	8475 2675 8700 2675
-$Comp
-L Device:CP C19
-U 1 1 5C296BC4
-P 7500 2850
-F 0 "C19" H 7618 2896 50  0000 L CNN
-F 1 "22uF" H 7618 2805 50  0000 L CNN
-F 2 "" H 7538 2700 50  0001 C CNN
-F 3 "~" H 7500 2850 50  0001 C CNN
-	1    7500 2850
-	1    0    0    -1
-$EndComp
 Wire Wire Line
 	7500 2675 7500 2700
@@
 Wire Wire Line
 	8300 4450 8300 4500
-$Comp
-L Device:CP C22
-U 1 1 5C2BBFDC
+Wire Wire Line
+	8300 4500 8525 4500
+Wire Wire Line
+	8725 4500 8725 4450
+Connection ~ 8300 4500
+Wire Wire Line
+	8300 4100 8300 4125
+Wire Wire Line
+	8300 4125 8725 4125
+Wire Wire Line
+	8725 4100 8725 4125
+Connection ~ 8300 4125
+Wire Wire Line
+	8300 4125 8300 4150
+Connection ~ 8725 4125
+Wire Wire Line
+	8725 4125 8725 4150
+Wire Wire Line
+	9125 4125 8725 4125
+Wire Wire Line
+	7800 4500 8300 4500
+Wire Wire Line
+	7725 3775 8125 3775
+Wire Wire Line
+	8725 3775 8725 3800
+Wire Wire Line
+	8500 3675 8500 3775
+Connection ~ 8500 3775
+Wire Wire Line
+	8500 3775 8725 3775
+Wire Wire Line
+	8300 3800 8300 3775
+Connection ~ 8300 3775
+Wire Wire Line
+	8300 3775 8500 3775
+Wire Wire Line
+	8125 3775 8125 3550
+Connection ~ 8125 3775
+Wire Wire Line
+	8125 3775 8300 3775
+Wire Wire Line
+	8525 4625 8525 4500
+Connection ~ 8525 4500
+Wire Wire Line
+	8525 4500 8725 4500
+$Comp
+L Device:C C18
+U 1 1 5C29211B
+P 8300 3950
+F 0 "C18" H 8415 3996 50  0000 L CNN
+F 1 "22u" H 8415 3905 50  0000 L CNN
+F 2 "" H 8338 3800 50  0001 C CNN
+F 3 "~" H 8300 3950 50  0001 C CNN
+	1    8300 3950
+	1    0    0    -1
+$EndComp
+$Comp
+L Device:C C21
+U 1 1 5C292362
+P 8725 3950
+F 0 "C21" H 8840 3996 50  0000 L CNN
+F 1 "22u" H 8840 3905 50  0000 L CNN
+F 2 "" H 8763 3800 50  0001 C CNN
+F 3 "~" H 8725 3950 50  0001 C CNN
+	1    8725 3950
+	1    0    0    -1
+$EndComp
+$Comp
+L Device:C C17
+U 1 1 5C2923C0
+P 8300 4300
+F 0 "C17" H 8415 4346 50  0000 L CNN
+F 1 "22u" H 8415 4255 50  0000 L CNN
+F 2 "" H 8338 4150 50  0001 C CNN
+F 3 "~" H 8300 4300 50  0001 C CNN
+	1    8300 4300
+	1    0    0    -1
+$EndComp
+$Comp
+L Device:C C22
+U 1 1 5C292428
 P 8725 4300
-F 0 "C22" H 8843 4346 50  0000 L CNN
-F 1 "22uF" H 8843 4255 50  0000 L CNN
+F 0 "C22" H 8840 4346 50  0000 L CNN
+F 1 "22u" H 8840 4255 50  0000 L CNN
 F 2 "" H 8763 4150 50  0001 C CNN
 F 3 "~" H 8725 4300 50  0001 C CNN
@@
 $EndComp
 $Comp
-L Device:CP C21
-U 1 1 5C2BC030
-P 8725 3950
-F 0 "C21" H 8843 3996 50  0000 L CNN
-F 1 "22uF" H 8843 3905 50  0000 L CNN
-F 2 "" H 8763 3800 50  0001 C CNN
-F 3 "~" H 8725 3950 50  0001 C CNN
-	1    8725 3950
-	1    0    0    -1
-$EndComp
-Wire Wire Line
-	8300 4500 8525 4500
-Wire Wire Line
-	8725 4500 8725 4450
-Connection ~ 8300 4500
-Wire Wire Line
-	8300 4100 8300 4125
-Wire Wire Line
-	8300 4125 8725 4125
-Wire Wire Line
-	8725 4100 8725 4125
-Connection ~ 8300 4125
-Wire Wire Line
-	8300 4125 8300 4150
-Connection ~ 8725 4125
-Wire Wire Line
-	8725 4125 8725 4150
-Wire Wire Line
-	9125 4125 8725 4125
-Wire Wire Line
-	7800 4500 8300 4500
-$Comp
-L Device:CP C18
-U 1 1 5C28145A
-P 8300 3950
-F 0 "C18" H 8418 3996 50  0000 L CNN
-F 1 "22uF" H 8418 3905 50  0000 L CNN
-F 2 "" H 8338 3800 50  0001 C CNN
-F 3 "~" H 8300 3950 50  0001 C CNN
-	1    8300 3950
-	1    0    0    -1
-$EndComp
-Wire Wire Line
-	7725 3775 8125 3775
-Wire Wire Line
-	8725 3775 8725 3800
-Wire Wire Line
-	8500 3675 8500 3775
-Connection ~ 8500 3775
-Wire Wire Line
-	8500 3775 8725 3775
-Wire Wire Line
-	8300 3800 8300 3775
-Connection ~ 8300 3775
-Wire Wire Line
-	8300 3775 8500 3775
-Wire Wire Line
-	8125 3775 8125 3550
-Connection ~ 8125 3775
-Wire Wire Line
-	8125 3775 8300 3775
-Wire Wire Line
-	8525 4625 8525 4500
-Connection ~ 8525 4500
-Wire Wire Line
-	8525 4500 8725 4500
+L Device:C C19
+U 1 1 5C29B778
+P 7500 2850
+F 0 "C19" H 7615 2896 50  0000 L CNN
+F 1 "22u" H 7615 2805 50  0000 L CNN
+F 2 "" H 7538 2700 50  0001 C CNN
+F 3 "~" H 7500 2850 50  0001 C CNN
+	1    7500 2850
+	1    0    0    -1
+$EndComp
+$Comp
+L Device:C C20
+U 1 1 5C29B7FA
+P 8475 2850
+F 0 "C20" H 8590 2896 50  0000 L CNN
+F 1 "22u" H 8590 2805 50  0000 L CNN
+F 2 "" H 8513 2700 50  0001 C CNN
+F 3 "~" H 8475 2850 50  0001 C CNN
+	1    8475 2850
+	1    0    0    -1
+$EndComp
 $EndSCHEMATC

Commit message: fixed incorrect chip number, assigned packages
Parts:
- C13, C14, C15, C16, C17, C18, C19, C20, C21, C22: footprint (none) -> Capacitor_SMD:C_0805_2012Metric_Pad1.33x1.40mm_HandSolder
- J1: footprint (none) -> Connector_PinHeader_2.54mm:PinHeader_1x04_P2.54mm_Vertical
- J2: footprint (none) -> Connector_PinHeader_2.54mm:PinHeader_1x09_P2.54mm_Vertical
- L1, L2, L3: footprint (none) -> Inductor_SMD:L_0603_1608Metric_Pad1.05x0.95mm_HandSolder
- P1: footprint (none) -> mta-156:MTA-156-4
- TR1, TR2: footprint (none) -> trim:trimmer
- U4: footprint (none) -> Package_SO:TSSOP-14_4.4x5mm_P0.65mm
- U5: footprint (none) -> Package_TO_SOT_SMD:SOT-89-3_Handsoldering
Changed lines of the file:
@@
 F 0 "U4" H 2150 4747 60  0000 C CNN
 F 1 "DAC8168" H 2150 4641 60  0000 C CNN
-F 2 "" H 2150 3800 60  0001 C CNN
+F 2 "Package_SO:TSSOP-14_4.4x5mm_P0.65mm" H 2150 3800 60  0001 C CNN
 F 3 "" H 2150 3800 60  0001 C CNN
 	1    2150 3700
@@
 F 0 "J2" H 2504 1517 50  0000 L CNN
 F 1 "cv out" H 2504 1426 50  0000 L CNN
-F 2 "" H 2425 1475 50  0001 C CNN
+F 2 "Connector_PinHeader_2.54mm:PinHeader_1x09_P2.54mm_Vertical" H 2425 1475 50  0001 C CNN
 F 3 "~" H 2425 1475 50  0001 C CNN
 	1    2425 1475
@@
 F 0 "J1" H 670 1817 50  0000 C CNN
 F 1 "digi in" H 670 1726 50  0000 C CNN
-F 2 "" H 750 1500 50  0001 C CNN
+F 2 "Connector_PinHeader_2.54mm:PinHeader_1x04_P2.54mm_Vertical" H 750 1500 50  0001 C CNN
 F 3 "~" H 750 1500 50  0001 C CNN
 	1    750  1500
@@
 F 0 "TR1" H 3217 5221 50  0000 L CNN
 F 1 "VREF TRIM" H 3217 5130 50  0000 L CNN
-F 2 "" H 3150 5175 50  0000 C CNN
+F 2 "trim:trimmer" H 3150 5175 50  0001 C CNN
 F 3 "" H 3150 5175 50  0000 C CNN
 	1    3150 5175
@@
 F 0 "TR2" H 3218 6671 50  0000 L CNN
 F 1 "BIAS TRIM" H 3218 6580 50  0000 L CNN
-F 2 "" H 3150 6625 50  0000 C CNN
+F 2 "trim:trimmer" H 3150 6625 50  0001 C CNN
 F 3 "" H 3150 6625 50  0000 C CNN
 	1    3150 6625
@@
 F 0 "C16" H 2990 6871 50  0000 L CNN
 F 1 "1u" H 2990 6780 50  0000 L CNN
-F 2 "" H 2913 6675 50  0001 C CNN
+F 2 "Capacitor_SMD:C_0805_2012Metric_Pad1.33x1.40mm_HandSolder" H 2913 6675 50  0001 C CNN
 F 3 "~" H 2875 6825 50  0001 C CNN
 	1    2875 6825
@@
 F 0 "C15" H 2990 5421 50  0000 L CNN
 F 1 "1u" H 2990 5330 50  0000 L CNN
-F 2 "" H 2913 5225 50  0001 C CNN
+F 2 "Capacitor_SMD:C_0805_2012Metric_Pad1.33x1.40mm_HandSolder" H 2913 5225 50  0001 C CNN
 F 3 "~" H 2875 5375 50  0001 C CNN
 	1    2875 5375
@@
 F 0 "C13" V 1048 2500 50  0000 C CNN
 F 1 "22u" V 1139 2500 50  0000 C CNN
-F 2 "" H 1338 2350 50  0001 C CNN
+F 2 "Capacitor_SMD:C_0805_2012Metric_Pad1.33x1.40mm_HandSolder" H 1338 2350 50  0001 C CNN
 F 3 "~" H 1300 2500 50  0001 C CNN
 	1    1300 2500
@@
 F 0 "C14" V 1048 2900 50  0000 C CNN
 F 1 "1u" V 1139 2900 50  0000 C CNN
-F 2 "" H 1338 2750 50  0001 C CNN
+F 2 "Capacitor_SMD:C_0805_2012Metric_Pad1.33x1.40mm_HandSolder" H 1338 2750 50  0001 C CNN
 F 3 "~" H 1300 2900 50  0001 C CNN
 	1    1300 2900
@@
 F 0 "L2" V 7388 3775 50  0000 C CNN
 F 1 "BEAD" V 7479 3775 50  0000 C CNN
-F 2 "" V 7555 3775 50  0001 C CNN
+F 2 "Inductor_SMD:L_0603_1608Metric_Pad1.05x0.95mm_HandSolder" V 7555 3775 50  0001 C CNN
 F 3 "~" H 7625 3775 50  0001 C CNN
 	1    7625 3775
@@
 F 0 "L1" V 7163 4500 50  0000 C CNN
 F 1 "BEAD" V 7254 4500 50  0000 C CNN
-F 2 "" V 7330 4500 50  0001 C CNN
+F 2 "Inductor_SMD:L_0603_1608Metric_Pad1.05x0.95mm_HandSolder" V 7330 4500 50  0001 C CNN
 F 3 "~" H 7400 4500 50  0001 C CNN
 	1    7400 4500
@@
 F 0 "P1" H 6819 4290 50  0000 C CNN
 F 1 "MTA-156-4" H 6819 4199 50  0000 C CNN
-F 2 "" H 6900 3925 50  0000 C CNN
+F 2 "mta-156:MTA-156-4" H 6900 3925 50  0001 C CNN
 F 3 "" H 6900 3925 50  0000 C CNN
 	1    6900 3925
@@
 F 0 "L3" V 6988 3250 50  0000 C CNN
 F 1 "BEAD" V 7079 3250 50  0000 C CNN
-F 2 "" V 7155 3250 50  0001 C CNN
+F 2 "Inductor_SMD:L_0603_1608Metric_Pad1.05x0.95mm_HandSolder" V 7155 3250 50  0001 C CNN
 F 3 "~" H 7225 3250 50  0001 C CNN
 	1    7225 3250
@@
 F 0 "U5" H 8000 3290 50  0000 C CNN
 F 1 "LD2981" H 8000 3199 50  0000 C CNN
-F 2 "" H 8000 2825 50  0001 C CNN
+F 2 "Package_TO_SOT_SMD:SOT-89-3_Handsoldering" H 8000 2825 50  0001 C CNN
 F 3 "" H 8000 2825 50  0001 C CNN
 	1    8000 2825
@@
 F 0 "C18" H 8415 3996 50  0000 L CNN
 F 1 "22u" H 8415 3905 50  0000 L CNN
-F 2 "" H 8338 3800 50  0001 C CNN
+F 2 "Capacitor_SMD:C_0805_2012Metric_Pad1.33x1.40mm_HandSolder" H 8338 3800 50  0001 C CNN
 F 3 "~" H 8300 3950 50  0001 C CNN
 	1    8300 3950
@@
 F 0 "C21" H 8840 3996 50  0000 L CNN
 F 1 "22u" H 8840 3905 50  0000 L CNN
-F 2 "" H 8763 3800 50  0001 C CNN
+F 2 "Capacitor_SMD:C_0805_2012Metric_Pad1.33x1.40mm_HandSolder" H 8763 3800 50  0001 C CNN
 F 3 "~" H 8725 3950 50  0001 C CNN
 	1    8725 3950
@@
 F 0 "C17" H 8415 4346 50  0000 L CNN
 F 1 "22u" H 8415 4255 50  0000 L CNN
-F 2 "" H 8338 4150 50  0001 C CNN
+F 2 "Capacitor_SMD:C_0805_2012Metric_Pad1.33x1.40mm_HandSolder" H 8338 4150 50  0001 C CNN
 F 3 "~" H 8300 4300 50  0001 C CNN
 	1    8300 4300
@@
 F 0 "C22" H 8840 4346 50  0000 L CNN
 F 1 "22u" H 8840 4255 50  0000 L CNN
-F 2 "" H 8763 4150 50  0001 C CNN
+F 2 "Capacitor_SMD:C_0805_2012Metric_Pad1.33x1.40mm_HandSolder" H 8763 4150 50  0001 C CNN
 F 3 "~" H 8725 4300 50  0001 C CNN
 	1    8725 4300
@@
 F 0 "C19" H 7615 2896 50  0000 L CNN
 F 1 "22u" H 7615 2805 50  0000 L CNN
-F 2 "" H 7538 2700 50  0001 C CNN
+F 2 "Capacitor_SMD:C_0805_2012Metric_Pad1.33x1.40mm_HandSolder" H 7538 2700 50  0001 C CNN
 F 3 "~" H 7500 2850 50  0001 C CNN
 	1    7500 2850
@@
 F 0 "C20" H 8590 2896 50  0000 L CNN
 F 1 "22u" H 8590 2805 50  0000 L CNN
-F 2 "" H 8513 2700 50  0001 C CNN
+F 2 "Capacitor_SMD:C_0805_2012Metric_Pad1.33x1.40mm_HandSolder" H 8513 2700 50  0001 C CNN
 F 3 "~" H 8475 2850 50  0001 C CNN
 	1    8475 2850
