File: scale-offset.sch (KiCad schematic (older format))
At the start: 39 parts, among them U1 TL074, U2 TL074, U3 TL074

Commit message: no more F
Parts:
- C1, C2, C3, C4, C5, C6, C7, C8: value 100pF -> 100p
Changed lines of the file:
@@
 AR Path="/5C26D04F/5C26D33E" Ref="C1"  Part="1"
 F 0 "C1" V 1323 1150 50  0000 C CNN
-F 1 "100pF" V 1414 1150 50  0000 C CNN
+F 1 "100p" V 1414 1150 50  0000 C CNN
 F 2 "" H 1613 1000 50  0001 C CNN
 F 3 "~" H 1575 1150 50  0001 C CNN
@@
 AR Path="/5C26D04F/5C26D8ED" Ref="C2"  Part="1"
 F 0 "C2" V 1323 2550 50  0000 C CNN
-F 1 "100pF" V 1414 2550 50  0000 C CNN
+F 1 "100p" V 1414 2550 50  0000 C CNN
 F 2 "" H 1613 2400 50  0001 C CNN
 F 3 "~" H 1575 2550 50  0001 C CNN
@@
 AR Path="/5C26D04F/5C27023F" Ref="C3"  Part="1"
 F 0 "C3" V 1323 3950 50  0000 C CNN
-F 1 "100pF" V 1414 3950 50  0000 C CNN
+F 1 "100p" V 1414 3950 50  0000 C CNN
 F 2 "" H 1613 3800 50  0001 C CNN
 F 3 "~" H 1575 3950 50  0001 C CNN
@@
 AR Path="/5C26D04F/5C270279" Ref="C4"  Part="1"
 F 0 "C4" V 1323 5350 50  0000 C CNN
-F 1 "100pF" V 1414 5350 50  0000 C CNN
+F 1 "100p" V 1414 5350 50  0000 C CNN
 F 2 "" H 1613 5200 50  0001 C CNN
 F 3 "~" H 1575 5350 50  0001 C CNN
@@
 AR Path="/5C26D04F/5C271CB8" Ref="C5"  Part="1"
 F 0 "C5" V 3998 1150 50  0000 C CNN
-F 1 "100pF" V 4089 1150 50  0000 C CNN
+F 1 "100p" V 4089 1150 50  0000 C CNN
 F 2 "" H 4288 1000 50  0001 C CNN
 F 3 "~" H 4250 1150 50  0001 C CNN
@@
 AR Path="/5C26D04F/5C271CF2" Ref="C6"  Part="1"
 F 0 "C6" V 3998 2550 50  0000 C CNN
-F 1 "100pF" V 4089 2550 50  0000 C CNN
+F 1 "100p" V 4089 2550 50  0000 C CNN
 F 2 "" H 4288 2400 50  0001 C CNN
 F 3 "~" H 4250 2550 50  0001 C CNN
@@
 AR Path="/5C26D04F/5C271D2C" Ref="C7"  Part="1"
 F 0 "C7" V 3998 3950 50  0000 C CNN
-F 1 "100pF" V 4089 3950 50  0000 C CNN
+F 1 "100p" V 4089 3950 50  0000 C CNN
 F 2 "" H 4288 3800 50  0001 C CNN
 F 3 "~" H 4250 3950 50  0001 C CNN
@@
 AR Path="/5C26D04F/5C271D66" Ref="C8"  Part="1"
 F 0 "C8" V 3998 5350 50  0000 C CNN
-F 1 "100pF" V 4089 5350 50  0000 C CNN
+F 1 "100p" V 4089 5350 50  0000 C CNN
 F 2 "" H 4288 5200 50  0001 C CNN
 F 3 "~" H 4250 5350 50  0001 C CNN

Commit message: fixed incorrect chip number, assigned packages
Parts:
- C1, C10, C11, C12, C2, C3, C4, C5, C6, C7, C8, C9: footprint (none) -> Capacitor_SMD:C_0805_2012Metric_Pad1.33x1.40mm_HandSolder
- R1, R10, R11, R12, R13, R14, R15, R16, R17, R18, R19, R2, R20, R21, R22, R23, R24, R3, R4, R5, R6, R7, R8, R9: footprint (none) -> Resistor_SMD:R_0805_2012Metric_Pad1.33x1.40mm_HandSolder
- U1: renamed from U3; footprint (none) -> Package_SO:TSSOP-14_4.4x5mm_P0.65mm
- U1, U2: footprint (none) -> Package_SO:TSSOP-14_4.4x5mm_P0.65mm
