File: mod-dac.kicad_pcb (KiCad board)
At the start: 2 copper layers, 58 parts, among them J1 digi in, J2 cv out, P1 MTA-156-4, U1 TL074, U2 TL074, U4 DAC8168, U5 LD2981

Commit message: more rough layout work
Parts:
- moved C16 61.5 mm to (83.8, 105.9)
- moved TR2 61.5 mm to (82.9, 112.5)
- moved C14 59.5 mm to (88.9, 93.0), turned to 270 degrees
- moved C13 57.7 mm to (86.9, 93.0), turned to 270 degrees
- moved P1 55.2 mm to (95.3, 40.6), turned to 270 degrees
- moved U4 55.0 mm to (90.4, 86.9), turned to 90 degrees
- moved C9 54.8 mm to (105.9, 66.1), turned to 90 degrees
- moved C11 51.2 mm to (105.9, 93.0), turned to 90 degrees
- moved L2 49.2 mm to (93.8, 45.2), turned to 0 degrees
- moved L3 47.3 mm to (95.0, 48.8), turned to 270 degrees
- moved U1 46.5 mm to (105.9, 72.6), turned to 270 degrees
- moved C21 45.2 mm to (91.9, 47.2), turned to 180 degrees
- moved U2 44.5 mm to (105.9, 99.6), turned to 270 degrees
- moved J1 43.8 mm to (84.3, 81.8), turned to 0 degrees
- moved C18 42.0 mm to (91.9, 50.8), turned to 180 degrees
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Connections:
- R1 pad 2: dac0 -> dac1
- R13 pad 2: dac4 -> dac6
- R14 pad 2: dac5 -> dac4
- R15 pad 2: dac6 -> dac2
- R16 pad 2: dac7 -> dac0
- R2 pad 2: dac1 -> dac3
- R3 pad 2: dac2 -> dac5
- R4 pad 2: dac3 -> dac7

Commit message: more routing
Parts:
- added REF**: MountingHole_3.2mm_M3, MountingHole:MountingHole_3.2mm_M3, F.Cu at (122.6, 58.8)
- added REF**: MountingHole_3.2mm_M3, MountingHole:MountingHole_3.2mm_M3, F.Cu at (123.6, 111.4)
- added REF**: MountingHole_3.2mm_M3, MountingHole:MountingHole_3.2mm_M3, F.Cu at (86.1, 111.4)
- added REF**: MountingHole_3.2mm_M3, MountingHole:MountingHole_3.2mm_M3, F.Cu at (86.0, 58.9)
- moved TR2 32.6 mm to (102.4, 86.4), turned to 90 degrees
- moved C16 23.7 mm to (95.8, 85.5), turned to 90 degrees
- moved C15 22.4 mm to (90.6, 98.6)
- moved TR1 22.4 mm to (89.6, 104.9)
- moved P1 20.9 mm to (104.1, 59.6)
- moved L2 20.2 mm to (101.1, 64.0)
- moved L1 19.8 mm to (89.9, 63.8)
- moved C19 18.9 mm to (84.1, 73.7), turned to 270 degrees
- moved L3 18.2 mm to (101.1, 65.9), turned to 180 degrees
- moved C17 18.1 mm to (93.6, 64.0)
- moved C22 17.8 mm to (93.6, 67.3)
- moved C21 17.6 mm to (97.3, 64.0)
- moved C18 17.4 mm to (97.3, 67.3)
- moved C20 16.9 mm to (92.7, 73.7), turned to 270 degrees
- moved U5 15.7 mm to (88.6, 73.7), turned to 270 degrees
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Connections:
- J1 pad 2: \SYNC -> DIN
- J1 pad 3: DIN -> \SYNC
Routing:
- net REFVCC: track 0.00 -> 43.2 mm, vias 0 -> 2
- net Net-(C19-Pad1): track 0.00 -> 21.2 mm, vias 0 -> 2
- net Net-(C8-Pad2): track 0.00 -> 20.7 mm, vias 0 -> 2
- net Net-(C4-Pad2): track 0.00 -> 20.4 mm, vias 0 -> 2
- net Net-(C6-Pad2): track 0.00 -> 20.0 mm
- net Net-(C5-Pad2): track 0.00 -> 19.9 mm, vias 0 -> 2
- net Net-(C1-Pad2): track 0.00 -> 19.9 mm, vias 0 -> 2
- net Net-(C7-Pad2): track 0.00 -> 19.8 mm
- net vout0: track 0.00 -> 19.6 mm
- net vout7: track 0.00 -> 19.5 mm
- net Net-(C2-Pad2): track 0.00 -> 19.5 mm
- net Net-(C3-Pad2): track 0.00 -> 19.0 mm
- net dac1: track 0.00 -> 18.2 mm
- net dac0: track 0.00 -> 17.7 mm
- net Net-(C6-Pad1): track 0.00 -> 16.8 mm
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
Commit message: i think i've routed the rest of the non gnd signals
Parts:
- C10, C11, C12, C9: moved to B.Cu
Routing:
- net vbias: track 4.12 -> 58.5 mm, vias 0 -> 5
- net -15V: track 10.5 -> 56.5 mm, vias 0 -> 3
- net +15V: track 10.9 -> 47.2 mm, vias 0 -> 3
- net vref: track 0.00 -> 18.3 mm, vias 0 -> 1
- net REFVCC: track 43.2 -> 55.0 mm
- net Net-(C6-Pad2): track 20.0 -> 21.2 mm
- net Net-(C3-Pad2): track 19.0 -> 20.1 mm
- net Net-(C7-Pad2): track 19.8 -> 20.8 mm
- net Net-(C1-Pad2): track 19.9 -> 20.8 mm, vias 2 -> 0
- net Net-(C2-Pad2): track 19.5 -> 20.4 mm
- net Net-(C3-Pad1): track 16.2 -> 17.0 mm
- net Net-(C6-Pad1): track 16.8 -> 17.4 mm
- net Net-(C19-Pad1): track 21.2 -> 20.7 mm
- net Net-(C4-Pad2): track 20.4 -> 20.7 mm, vias 2 -> 0
- net Net-(C5-Pad2): track 19.9 -> 20.2 mm, vias 2 -> 0
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
Commit message: edge cut
Parts:
- removed REF**: MountingHole_3.2mm_M3, MountingHole:MountingHole_3.2mm_M3
- added REF1: MountingHole_3.2mm_M3, MountingHole:MountingHole_3.2mm_M3, F.Cu at (85.9, 58.9)
- moved REF4 0.65 mm to (122.9, 111.3)
- moved REF2 0.40 mm to (122.9, 58.9)
- moved REF3 0.28 mm to (85.9, 111.3)
- renumbered REF** to REF2, REF** to REF3, REF** to REF4
Other:
- board outline added: 44.2 x 59.4 mm
Changed lines of the file:
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@@
   (general
     (thickness 1.6)
-    (drawings 0)
+    (drawings 1)
     (tracks 364)
     (zones 0)
@@
   )
   (module MountingHole:MountingHole_3.2mm_M3 (layer F.Cu)
-    (at 122.555 58.801)
+    (at 122.936 58.928)
     (descr "Mounting Hole 3.2mm, no annular, M3")
     (tags "mounting hole 3.2mm no annular m3")
     (attr virtual)
-    (fp_text reference REF** (at 0 -4.2) (layer F.SilkS)
+    (fp_text reference REF2 (at 0 -4.2) (layer F.Fab) hide
       (effects (font (size 1 1) (thickness 0.15)))
     )
@@
   )
   (module MountingHole:MountingHole_3.2mm_M3 (layer F.Cu)
-    (at 123.571 111.379)
+    (at 122.936 111.252)
     (descr "Mounting Hole 3.2mm, no annular, M3")
     (tags "mounting hole 3.2mm no annular m3")
     (attr virtual)
-    (fp_text reference REF** (at 0 -4.2) (layer F.SilkS)
+    (fp_text reference REF4 (at 0 -4.2) (layer F.Fab) hide
       (effects (font (size 1 1) (thickness 0.15)))
     )
@@
   )
   (module MountingHole:MountingHole_3.2mm_M3 (layer F.Cu)
-    (at 86.106 111.379)
+    (at 85.852 111.252)
     (descr "Mounting Hole 3.2mm, no annular, M3")
     (tags "mounting hole 3.2mm no annular m3")
     (attr virtual)
-    (fp_text reference REF** (at 0 -4.2) (layer F.SilkS)
+    (fp_text reference REF3 (at 0 -4.2) (layer F.Fab) hide
       (effects (font (size 1 1) (thickness 0.15)))
     )
@@
   )
   (module MountingHole:MountingHole_3.2mm_M3 (layer F.Cu)
-    (at 85.979 58.928)
+    (at 85.852 58.928)
     (descr "Mounting Hole 3.2mm, no annular, M3")
     (tags "mounting hole 3.2mm no annular m3")
     (attr virtual)
-    (fp_text reference REF** (at 0 -4.2) (layer F.SilkS)
+    (fp_text reference REF1 (at 0 -4.2) (layer F.Fab) hide
       (effects (font (size 1 1) (thickness 0.15)))
     )
@@
     (pad 1 np_thru_hole circle (at 0 0) (size 3.2 3.2) (drill 3.2) (layers *.Cu *.Mask))
   )
+  (gr_poly (pts (xy 82.296 55.372) (xy 126.492 55.372) (xy 126.492 114.808) (xy 82.296 114.808)) (layer Edge.Cuts) (width 0.15))
   (segment (start 114.457 61.722) (end 114.457 63.754) (width 0.254) (layer F.Cu) (net 1))
   (segment (start 112.179 63.754) (end 107.218 68.715) (width 0.254) (layer F.Cu) (net 1))

Commit message: moved power a bit
Parts:
- moved P1 4.45 mm to (108.5, 59.6)
Routing:
- net GND: track 12.9 -> 22.5 mm
- net Net-(L2-Pad2): track 7.22 -> 12.0 mm
- net Net-(L1-Pad2): track 6.46 -> 9.30 mm
- added copper zone on B.Cu, net GND
- added copper zone on F.Cu, net GND
Changed lines of the file:
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@@
     (thickness 1.6)
     (drawings 1)
-    (tracks 364)
+    (tracks 369)
     (zones 0)
     (modules 62)
@@
   )
   (setup
-    (last_trace_width 0.254)
+    (last_trace_width 0.4064)
     (user_trace_width 0.254)
     (user_trace_width 0.4064)
@@
     (pad_to_mask_clearance 0.2)
     (aux_axis_origin 0 0)
-    (visible_elements FFFFFF7F)
+    (visible_elements FFFFF77F)
     (pcbplotparams
       (layerselection 0x010fc_ffffffff)
@@
   )
   (module mta-156:MTA-156-4 (layer F.Cu)
-    (at 104.059 59.563 270)
+    (at 108.504 59.563 270)
     (descr MTA-156-4)
     (tags MTA-156-4)
@@
   (segment (start 99.162499 84.5335) (end 99.862 83.833999) (width 0.4064) (layer F.Cu) (net 18))
   (segment (start 95.758 84.5335) (end 99.162499 84.5335) (width 0.4064) (layer F.Cu) (net 18))
-  (segment (start 96.139 59.563) (end 100.099 59.563) (width 0.4064) (layer F.Cu) (net 18))
-  (segment (start 96.139 63.754) (end 96.393 64.008) (width 0.4064) (layer F.Cu) (net 18))
-  (segment (start 96.139 59.563) (end 96.139 63.754) (width 0.4064) (layer F.Cu) (net 18))
+  (segment (start 104.544 59.563) (end 100.584 59.563) (width 0.4064) (layer F.Cu) (net 18))
+  (segment (start 97.070674 63.330326) (end 96.393 64.008) (width 0.4064) (layer F.Cu) (net 18))
+  (segment (start 97.070674 62.949326) (end 97.070674 63.330326) (width 0.4064) (layer F.Cu) (net 18))
+  (segment (start 97.5506 62.4694) (end 97.070674 62.949326) (width 0.4064) (layer F.Cu) (net 18))
+  (segment (start 98.9276 62.4694) (end 97.5506 62.4694) (width 0.4064) (layer F.Cu) (net 18))
+  (segment (start 100.584 59.563) (end 100.584 60.813) (width 0.4064) (layer F.Cu) (net 18))
+  (segment (start 100.584 60.813) (end 98.9276 62.4694) (width 0.4064) (layer F.Cu) (net 18))
+  (segment (start 96.393 64.008) (end 94.488 64.008) (width 0.4064) (layer F.Cu) (net 18))
+  (segment (start 94.488 64.008) (end 94.488 67.31) (width 0.4064) (layer F.Cu) (net 18))
+  (segment (start 94.488 67.31) (end 96.393 67.31) (width 0.4064) (layer F.Cu) (net 18))
   (segment (start 91.059 64.008) (end 90.805 63.754) (width 0.4064) (layer F.Cu) (net 19))
   (segment (start 92.613 64.008) (end 91.059 64.008) (width 0.4064) (layer F.Cu) (net 19))
@@
   (segment (start 123.952 94.615) (end 122.047 96.52) (width 0.254) (layer F.Cu) (net 34))
   (segment (start 122.047 96.52) (end 122.047 106.045) (width 0.254) (layer F.Cu) (net 34))
-  (segment (start 89.055 63.179) (end 89.055 63.754) (width 0.4064) (layer F.Cu) (net 35))
-  (segment (start 90.5226 59.563) (end 89.055 61.0306) (width 0.4064) (layer F.Cu) (net 35))
-  (segment (start 89.055 61.0306) (end 89.055 63.179) (width 0.4064) (layer F.Cu) (net 35))
-  (segment (start 92.179 59.563) (end 90.5226 59.563) (width 0.4064) (layer F.Cu) (net 35))
-  (segment (start 101.981 63.433) (end 101.981 64.008) (width 0.4064) (layer F.Cu) (net 36))
-  (segment (start 101.981 62.891) (end 101.981 63.433) (width 0.4064) (layer F.Cu) (net 36))
-  (segment (start 104.059 60.813) (end 101.981 62.891) (width 0.4064) (layer F.Cu) (net 36))
-  (segment (start 104.059 59.563) (end 104.059 60.813) (width 0.4064) (layer F.Cu) (net 36))
+  (segment (start 93.246 59.563) (end 89.055 63.754) (width 0.4064) (layer F.Cu) (net 35))
+  (segment (start 96.624 59.563) (end 93.246 59.563) (width 0.4064) (layer F.Cu) (net 35))
   (segment (start 101.981 65.885) (end 101.953 65.913) (width 0.4064) (layer F.Cu) (net 36))
   (segment (start 101.981 64.008) (end 101.981 65.885) (width 0.4064) (layer F.Cu) (net 36))
+  (segment (start 106.9654 64.008) (end 102.606 64.008) (width 0.4064) (layer F.Cu) (net 36))
+  (segment (start 102.606 64.008) (end 101.981 64.008) (width 0.4064) (layer F.Cu) (net 36))
+  (segment (start 108.504 62.4694) (end 106.9654 64.008) (width 0.4064) (layer F.Cu) (net 36))
+  (segment (start 108.504 59.563) (end 108.504 62.4694) (width 0.4064) (layer F.Cu) (net 36))
   (segment (start 98.552 102.87) (end 99.3925 102.87) (width 0.254) (layer F.Cu) (net 37))
   (segment (start 98.298 102.87) (end 98.552 102.87) (width 0.254) (layer F.Cu) (net 37))
@@
   (segment (start 99.725 75.692) (end 97.79 75.692) (width 0.254) (layer F.Cu) (net 44))
   (segment (start 97.79 75.692) (end 92.374 81.108) (width 0.254) (layer F.Cu) (net 44))
+  (zone (net 18) (net_name GND) (layer B.Cu) (hatch edge 0.508)
+    (connect_pads (clearance 0.508))
+    (min_thickness 0.254)
+    (fill yes (arc_segments 16) (thermal_gap 0.508) (thermal_bridge_width 0.508))
+    (polygon
+      (pts
+        (xy 82.296 55.372) (xy 126.492 55.372) (xy 126.492 114.808) (xy 82.296 114.808)
+      )
+    )
+  )
+  (zone (net 18) (net_name GND) (layer F.Cu) (hatch edge 0.508)
+    (connect_pads (clearance 0.508))
+    (min_thickness 0.254)
+    (fill yes (arc_segments 16) (thermal_gap 0.508) (thermal_bridge_width 0.508))
+    (polygon
+      (pts
+        (xy 82.296 55.372) (xy 126.492 55.372) (xy 126.492 114.808) (xy 82.296 114.808)
+      )
+    )
+  )
 )
